File: v3/hardware/BigCoilBoard.kicad_sch (KiCad schematic)
At the start: 141 parts, among them J1 Conn_01x02, J10 PFC_OUT, J11 THERM2_IN, J12 THERM3_IN, J13 THERM4_IN, J14 THERM5_IN, J16 Conn_ARM_JTAG_SWD_10, J17 Conn_01x04, J18 Conn_01x04, J19 Conn_01x04, J2 Conn_01x02, J20 Screw_Terminal_01x01, J21 Screw_Terminal_01x01, J22 Screw_Terminal_01x01, J23 Screw_Terminal_01x01, J24 Conn_01x04, J3 Conn_01x03_Pin, J5 THERM1_IN, J6 Conn_01x03_Pin, J7 Conn_01x04, J8 CONTACTOR_1, J9 CONTACTOR_2, K1 G5NB-1A-DC24, K2 G5NB-1A-DC24, Q1 T2N7002AK, Q2 T2N7002AK, Q3 T2N7002AK, Q4 T2N7002AK, Q5 T2N7002AK, Q6 T2N7002AK, Q7 T2N7002AK, U1 STM32G474CBTx, U10 IF-D95, U11 IF-E96E, U12 LD1117S33TR_SOT223, U13 TC7662Bx0A, U14 L7812, U2 MCP6477-E/SN, U3 CSTNE8M00G550000R0, U4 STM32G473RBTx, U6 MGJ2D241709SC, U7 STGAP2SM, U8 SN74LV1T34DBV, U9 IF-D95

Commit message: v3 work, implemented dcm pfc in v2
Parts:
- removed C26, C32, C34, C36: 0.1u, Capacitor_SMD:C_0805_2012Metric, symbol Device:C
- removed C33: 4.7u, Capacitor_SMD:C_0805_2012Metric, symbol Device:C
- removed C35, C37: 330u, Library:860020575013, symbol Device:C_Polarized
- removed J1: Conn_01x02, Connector_PinSocket_2.54mm:PinSocket_1x02_P2.54mm_Vertical, symbol Connector_Generic:Conn_01x02
- removed J16: Conn_ARM_JTAG_SWD_10, Connector_PinHeader_1.27mm:PinHeader_2x05_P1.27mm_Vertical, symbol Connector:Conn_ARM_JTAG_SWD_10
- removed J3, J6: Conn_01x03_Pin, Connector_PinSocket_2.54mm:PinSocket_1x03_P2.54mm_Vertical, symbol Connector:Conn_01x03_Pin
- removed TP2, TP3, TP4, TP5, TP6: TestPoint, TestPoint:TestPoint_Pad_2.0x2.0mm, symbol Connector:TestPoint
- removed U1: STM32G474CBTx, Package_QFP:LQFP-48_7x7mm_P0.5mm, symbol MCU_ST_STM32G4:STM32G474CBTx
- removed U13: TC7662Bx0A, Package_SO:SOIC-8_3.9x4.9mm_P1.27mm, symbol Converter_DCDC:TC7662Bx0A
- removed U14: L7812, Package_TO_SOT_THT:TO-220-3_Vertical, symbol Regulator_Linear:L7812
- removed U3: CSTNE8M00G550000R0, Crystal:Resonator_SMD_Murata_CSTxExxV-3Pin_3.0x1.1mm, symbol New_Library:CSTNE8M00G550000R0
- removed U7: STGAP2SM, Package_SO:SOIC-8_3.9x4.9mm_P1.27mm, symbol Driver_FET:STGAP2SM
- removed U8: SN74LV1T34DBV, Package_TO_SOT_SMD:SOT-23-5, symbol Logic_LevelTranslator:SN74LV1T34DBV
- added C24: 1n, Capacitor_SMD:C_0805_2012Metric, symbol Device:C
- added C7: 0.1u, Capacitor_SMD:C_0805_2012Metric, symbol Device:C
- added IC1: IXDI630YI, Package_TO_SOT_SMD:TO-263-5_TabPin6, symbol New_Library:IXDI630YI
- added Q8: T2N7002AK, Package_TO_SOT_SMD:SOT-23, symbol Transistor_FET:T2N7002AK
- added R35, R36, R37, R38, R39, R40: 10k, Resistor_SMD:R_0805_2012Metric, symbol Device:R
- added U1, U3: SQJ500AEP-T1_GE3, Library:SQJ500AEP-T1_GE3_VIS, symbol New_Library:SQJ500AEP-T1_GE3
- added U5: MCP6477-E/SN, Package_SO:SOIC-8_3.9x4.9mm_P1.27mm, symbol Amplifier_Operational:MCP6002-xSN
- added U8: 6N136S, Package_DIP:SMDIP-8_W9.53mm, symbol Isolator:6N136S
- added Y2: CSTNE8M00G550000R0, Crystal:Resonator_SMD_Murata_CSTxExxV-3Pin_3.0x1.1mm, symbol Device:Resonator
- R22: value 13R? -> 1k; footprint Resistor_THT:R_Axial_DIN0207_L6.3mm_D2.5mm_P10.16mm_Horizontal -> Resistor_SMD:R_0805_2012Metric
- R23: value 1k -> 10k
- R4: value 0R -> 120R; footprint Resistor_SMD:R_1210_3225Metric -> Resistor_SMD:R_0805_2012Metric
- R5: value 0R -> 1R; footprint Resistor_SMD:R_1210_3225Metric -> Resistor_THT:R_Axial_DIN0207_L6.3mm_D2.5mm_P10.16mm_Horizontal
Connections:
- net +12V is gone; now on net GND: J24.3 (Pin_3)
- net +3.3V: now also R4.2
- net +5V: now also J24.4 (Pin_4)
- net 0V_ISO: now also C7.1, R35.2, U8.8
- net BOOT0: now also U4.61 (PB8)
- net B_LED1: now also U4.52 (PC10)
- net B_LED2: now also U4.53 (PC11)
- net B_LED3: now also U4.54 (PC12)
- net CN1: now also U4.2 (PC13)
- net CN2: now also U4.3 (PC14)
- net GND: now also R23.2, C24.1, Q8.2 (S), R39.2, Y2.2; no longer J24.4 (Pin_4), R22.2
- net INT_IN: now also U4.24 (PB0), U4.25 (PB1)
- net I_L: now also U4.33 (PB11); no longer C38.2, R23.1
- net LED1: now also U4.57 (PB4)
- net LED2: now also U4.58 (PB5)
- net LED3: now also U4.59 (PB6)
- net LED4: now also U4.60 (PB7)
- net NRST: now also U4.7 (PG10)
- net PFC: now also U4.38 (PC6), Q8.1 (G)
- net THERM1: now also U4.8 (PC0)
- net THERM2: now also U4.9 (PC1)
- net THERM3: now also U4.10 (PC2)
- net THERM4: now also U4.11 (PC3)
- net THERM5: now also U4.12 (PA0)
- net UART_RX: now also U4.23 (PC5)
- net UART_TX: now also U4.22 (PC4)
- net V24_SENSE: now also U4.43 (PA9)
- net VAC_SENSE: now also U4.34 (PB12)
- net VBUS_SENSE: now also U4.35 (PB13)
- net V-_ISO: now reaches C3.2, C6.2, U6.5 (-VOUT)
- net V-_ISO: now also C7.2, IC1.3 (GND_1), IC1.6 (GND_2), IC1.7 (GND_3), U8.5
- net at J10.1 (Pin_1), R5.2: no longer R4.2
- net V+_ISO: now reaches C1.1, C2.1, U6.7 (+VOUT)
- net V+_ISO: now also IC1.1 (VCC)
- net at R5.1: now also IC1.2 (~{OUT})
- net at R4.1: now also U8.2
- net OCD_COMP: now reaches U4.13 (PA1)
- net IN+: now reaches U4.17 (PA3)
- net IN-: now reaches U4.19 (PA5)
- net VREF: now reaches U4.28 (VREF+)
- net GD_OUT: now reaches U4.40 (PC8)
- net GD_EN: now reaches U4.41 (PC9)
- net USB_D-: now reaches U4.45 (PA11)
- net USB_D+: now reaches U4.46 (PA12)
- net DIO: now reaches U4.49 (PA13)
- net at U4.5 (PF0): now also Y2.1
- net CLK: now reaches U4.50 (PA14)
- net SWO: now reaches U4.56 (PB3)
- net at U4.6 (PF1): now also Y2.3
- net -12V renamed I_L_REF
- net I_L_REF: now also C24.2, R36.1
- new net: Q8.3 (D), U8.3
- new net: J24.2 (Pin_2), R22.2, R23.1
- new net: R38.1, U5.1, U5.2 (-)
- new net: R38.2, R39.1, U5.5 (+)
- new net: IC1.4 (IN), R35.1, U8.6
- new net: R36.2, R37.1, U5.6 (-)
- new net: C38.2, R22.1, U5.3 (+)
- new net: R37.2, R40.1, U5.7
- no-connect marks 5 -> 1
Other:
- moved on the sheet: C38, D3, J10, J24, R23, U4
